Commit message: Add letter task

File: environments/suction/suction-head.urdf (robot description, URDF)
Before this commit: robot suction-head.urdf, 2 links, 1 joints
Links:
- link tipLink: geometry collision cylinder length=0.028 radius=0.00001; visual mesh filename=tip.obj scale=0.001 0.001 0.001

Commit message: update a lot

File: environments/suction/suction-head.urdf (robot description, URDF)
Before this commit: robot suction-head.urdf, 2 links, 1 joints
Links:
- link tipLink: geometry collision cylinder length=0.028 radius=0.005; visual mesh filename=tip.obj scale=0.001 0.001 0.001
